File: Hardware/Pro_Micro.sch (EAGLE design)
At the start: 33 parts, among them U2 MIC5219, U3 ATMEGA32U4, Y1 16MHz

Commit message: Updated to current library parts with correct labels.  Changed silk to vector font. Moved a few bits of silk to not be over vias. Aligned angled traces to 45 degrees
Parts:
- U3: device Testing:ATMEGA32U4OUTFAKES -> SparkFun-DigitalIC:ATMEGA32U41:1-LESS_PASTE
Connections:
- net D14 renamed D17
Other:
- moved on the sheet: R2, R5, R7
